File: hardware/Ra-01_Handy_Neo/Ra-01_Handy_Neo.kicad_pcb (KiCad board)
At the start: 4 copper layers, 68.6 x 53.3 mm, 35 parts, among them J1 Power, J2 Digital/PWM, J3 Analog, J4 Digital/PWM, J5 Conn_Coaxial, J6 Conn_01x04_Pin, SW1 SW_Push, SW10 SW_Push, SW11 SW_Push, SW12 SW_Push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

Commit message: change designs
Routing:
- net GND: track 11.7 -> 11.9 mm, vias 0 -> 260
Other:
- board text added: "3V3"
- board text added: "For SPRESENSE extension boards only"
- board text added: "GND"
- board text added: "Ra-01"
- board text added: "Ra-01_Handy_Neo v1.0 Kazuma Kurokawa / k42uma"
- board text added: "SCL"
- board text added: "SDA"
- board text added: "電波めっちゃ出るよ〜〜"
