File: hardware/Ra-01_Handy_Neo/Ra-01_Handy_Neo.kicad_sch (KiCad schematic)
At the start: 0 parts

Commit message: add buttons and ra01 to sch
Parts:
- added J1: Power, Connector_PinSocket_2.54mm:PinSocket_1x08_P2.54mm_Vertical, symbol Connector_Generic:Conn_01x08
- added J2: Digital/PWM, Connector_PinSocket_2.54mm:PinSocket_1x10_P2.54mm_Vertical, symbol Connector_Generic:Conn_01x10
- added J3: Analog, Connector_PinSocket_2.54mm:PinSocket_1x06_P2.54mm_Vertical, symbol Connector_Generic:Conn_01x06
- added J4: Digital/PWM, Connector_PinSocket_2.54mm:PinSocket_1x08_P2.54mm_Vertical, symbol Connector_Generic:Conn_01x08
- added J5: Conn_Coaxial, Connector_Coaxial:SMA_BAT_Wireless_BWSMA-KWE-Z001, symbol Connector:Conn_Coaxial
- added R1, R10, R11, R12, R13, R2, R3, R4, R5, R6, R7, R8, R9: 10k, symbol Device:R
- added SW1, SW10, SW11, SW12, SW13, SW2, SW3, SW4, SW5, SW6, SW7, SW8, SW9: SW_Push, symbol Switch:SW_Push
- added U1: Ai-Thinker-Ra-01, RF_Module:Ai-Thinker-Ra-01-LoRa, symbol RF_Module:Ai-Thinker-Ra-01
- added U2, U3: 74HC165, symbol 74xx:74HC165
Connections:
- new net: U2.9 (Q7), U3.10 (DS)
- new net: J5.1 (In), U1.1 (ANT)
- new net *10: J2.8 (Pin_8)
- new net *9: J2.9 (Pin_9)
- new net +3V3: J1.4 (Pin_4), R1.1, R10.1, R11.1, R12.1, R13.1, R2.1, R3.1, R4.1, R5.1, R6.1, R7.1, R8.1, R9.1, U1.3 (VDD), U2.16 (VCC), U3.16 (VCC)
- new net +5V: J1.5 (Pin_5)
- new net A0: J3.1 (Pin_1)
- new net A1: J3.2 (Pin_2)
- new net A2: J3.3 (Pin_3)
- new net A3: J3.4 (Pin_4)
- new net AREF: J2.3 (Pin_3)
- new net CLK: J2.5 (Pin_5), U1.12 (SCK)
- new net CP: J4.2 (Pin_2), U2.2 (CP), U3.2 (CP)
- new net GND: J1.6 (Pin_6), J1.7 (Pin_7), J2.4 (Pin_4), J5.2 (Ext), SW1.1, SW10.1, SW11.1, SW12.1, SW13.1, SW2.1, SW3.1, SW4.1, SW5.1, SW6.1, SW7.1, SW8.1, SW9.1, U1.16 (GND), U1.2 (GND), U1.4 (~{RESET}), U1.9 (GND), U2.10 (DS), U2.15 (~{CE}), U2.8 (GND), U3.15 (~{CE}), U3.4 (D5), U3.5 (D6), U3.6 (D7), U3.8 (GND)
- new net IOREF: J1.2 (Pin_2)
- new net MISO: J2.6 (Pin_6), U1.13 (MISO)
- new net MOSI: J2.7 (Pin_7), U1.14 (MOSI)
- new net RX/0: J4.8 (Pin_8)
- new net Ra_CS: J2.10 (Pin_10), U1.15 (~{NSS})
- new net Ra_DIO0: J4.6 (Pin_6), U1.5 (DIO0)
- new net Ra_DIO1: J4.5 (Pin_5), U1.6 (DIO1)
- new net Ra_DIO2: J4.4 (Pin_4), U1.7 (DIO2)
- new net SCL/A5: J2.1 (Pin_1), J3.6 (Pin_6)
- new net SDA/A4: J2.2 (Pin_2), J3.5 (Pin_5)
- new net SO: J4.3 (Pin_3), U3.9 (Q7)
- new net SW0: R1.2, SW1.2, U2.11 (D0)
- new net SW1: R2.2, SW2.2, U2.12 (D1)
- new net SW2: R3.2, SW3.2, U2.13 (D2)
- new net SW3: R4.2, SW4.2, U2.14 (D3)
- new net SW4: R5.2, SW5.2, U2.3 (D4)
- new net SW5: R6.2, SW6.2, U2.4 (D5)
- new net SW6: R7.2, SW7.2, U2.5 (D6)
- new net SW7: R8.2, SW8.2, U2.6 (D7)
- new net SW8: R9.2, SW9.2, U3.11 (D0)
- new net SW9: R10.2, SW10.2, U3.12 (D1)
- new net SWB: R11.2, SW11.2, U3.13 (D2)
- new net SWE: R12.2, SW12.2, U3.14 (D3)
- new net SWS: R13.2, SW13.2, U3.3 (D4)
- new net TX/1: J4.7 (Pin_7)
- new net VCC: J1.8 (Pin_8)
- new net ~{PL}: J4.1 (Pin_1), U2.1 (~{PL}), U3.1 (~{PL})
- new net ~{RESET}: J1.3 (Pin_3)
- no-connect marks 0 -> 6
Other:
- note added: "* Indicates a PWM-capable pin"

Commit message: 80% done
Parts:
- added J6: Conn_01x04_Pin, Connector_PinHeader_2.54mm:PinHeader_1x04_P2.54mm_Horizontal, symbol Connector:Conn_01x04_Pin
- R1, R10, R11, R12, R13, R2, R3, R4, R5, R6, R7, R8, R9: footprint (none) -> Resistor_SMD:R_0603_1608Metric_Pad0.98x0.95mm_HandSolder
- SW1, SW10, SW11, SW12, SW13, SW2, SW3, SW4, SW5, SW6, SW7, SW8, SW9: footprint (none) -> Button_Switch_THT:SW_PUSH_6mm_H5mm
- U2, U3: value 74HC165 -> TC74HC165AF; footprint (none) -> Package_SO:JEITA_SOIC-16_3.9x9.9mm_P1.27mm
Connections:
- net *9 is gone; now on net Ra_CS: J2.9 (Pin_9)
- net +3V3: now also J6.3 (Pin_3)
- net GND: now also U3.12 (D1), U3.13 (D2), U3.14 (D3), J6.4 (Pin_4); no longer U1.4 (~{RESET}), U3.4 (D5), U3.5 (D6), U3.6 (D7)
- net Ra_CS: no longer J2.10 (Pin_10)
- net Ra_DIO0: now also J4.4 (Pin_4); no longer J4.6 (Pin_6)
- net Ra_DIO2: now also J4.6 (Pin_6); no longer J4.4 (Pin_4)
- net SO: now also J4.1 (Pin_1); no longer J4.3 (Pin_3)
- net SW0: now also U2.13 (D2); no longer U2.11 (D0)
- net SW2: now also U2.11 (D0); no longer U2.13 (D2)
- net SW6: now also U2.6 (D7); no longer U2.5 (D6)
- net SW7: now also U2.5 (D6); no longer U2.6 (D7)
- net SW9: now also U3.5 (D6); no longer U3.12 (D1)
- net SWB: now also U3.6 (D7); no longer U3.13 (D2)
- net SWE: now also U3.4 (D5); no longer U3.14 (D3)
- net ~{PL}: now also J4.3 (Pin_3); no longer J4.1 (Pin_1)
- net SCL/A5 renamed A5
- net A5: no longer J2.1 (Pin_1)
- net SDA/A4 renamed A4
- net A4: no longer J2.2 (Pin_2)
- new net Ra_RESET: J2.10 (Pin_10), U1.4 (~{RESET})
- new net SCL: J2.1 (Pin_1), J6.2 (Pin_2)
- new net SDA: J2.2 (Pin_2), J6.1 (Pin_1)

Commit message: pcb almost complete
Parts:
- J1, J4: footprint Connector_PinSocket_2.54mm:PinSocket_1x08_P2.54mm_Vertical -> Connector_PinHeader_2.54mm:PinHeader_1x08_P2.54mm_Vertical
- J2: footprint Connector_PinSocket_2.54mm:PinSocket_1x10_P2.54mm_Vertical -> Connector_PinHeader_2.54mm:PinHeader_1x10_P2.54mm_Vertical
- J3: footprint Connector_PinSocket_2.54mm:PinSocket_1x06_P2.54mm_Vertical -> Connector_PinHeader_2.54mm:PinHeader_1x06_P2.54mm_Vertical
Changed lines of the file:
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@@
 			)
 		)
-		(property "Footprint" "Connector_PinSocket_2.54mm:PinSocket_1x08_P2.54mm_Vertical"
+		(property "Footprint" "Connector_PinHeader_2.54mm:PinHeader_1x08_P2.54mm_Vertical"
 			(at 52.07 40.64 0)
 			(effects
@@
 			)
 		)
-		(property "Footprint" "Connector_PinSocket_2.54mm:PinSocket_1x10_P2.54mm_Vertical"
+		(property "Footprint" "Connector_PinHeader_2.54mm:PinHeader_1x10_P2.54mm_Vertical"
 			(at 69.85 38.1 0)
 			(effects
@@
 			)
 		)
-		(property "Footprint" "Connector_PinSocket_2.54mm:PinSocket_1x06_P2.54mm_Vertical"
+		(property "Footprint" "Connector_PinHeader_2.54mm:PinHeader_1x06_P2.54mm_Vertical"
 			(at 52.07 66.04 0)
 			(effects
@@
 			)
 		)
-		(property "Footprint" "Connector_PinSocket_2.54mm:PinSocket_1x08_P2.54mm_Vertical"
+		(property "Footprint" "Connector_PinHeader_2.54mm:PinHeader_1x08_P2.54mm_Vertical"
 			(at 69.85 68.58 0)
 			(effects

Commit message: change footprints and 3dsymbols to export step file
Parts:
- J5: footprint Connector_Coaxial:SMA_BAT_Wireless_BWSMA-KWE-Z001 -> Connector_Coaxial:SMA_Connector_at_Honbu_3-1478978-1
- SW1, SW10, SW11, SW12, SW13, SW2, SW3, SW4, SW5, SW6, SW7, SW8, SW9: footprint Button_Switch_THT:SW_PUSH_6mm_H5mm -> Button_Switch_THT:SW_PUSH_6mm_H6.5mm
Changed lines of the file:
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@@
 			)
 		)
-		(property "Footprint" "Button_Switch_THT:SW_PUSH_6mm_H5mm"
+		(property "Footprint" "Button_Switch_THT:SW_PUSH_6mm_H6.5mm"
 			(at 236.22 134.62 0)
 			(effects
@@
 			)
 		)
-		(property "Footprint" "Button_Switch_THT:SW_PUSH_6mm_H5mm"
+		(property "Footprint" "Button_Switch_THT:SW_PUSH_6mm_H6.5mm"
 			(at 160.02 134.62 0)
 			(effects
@@
 			)
 		)
-		(property "Footprint" "Button_Switch_THT:SW_PUSH_6mm_H5mm"
+		(property "Footprint" "Button_Switch_THT:SW_PUSH_6mm_H6.5mm"
 			(at 146.05 134.62 0)
 			(effects
@@
 			)
 		)
-		(property "Footprint" "Button_Switch_THT:SW_PUSH_6mm_H5mm"
+		(property "Footprint" "Button_Switch_THT:SW_PUSH_6mm_H6.5mm"
 			(at 223.52 134.62 0)
 			(effects
@@
 			)
 		)
-		(property "Footprint" "Button_Switch_THT:SW_PUSH_6mm_H5mm"
+		(property "Footprint" "Button_Switch_THT:SW_PUSH_6mm_H6.5mm"
 			(at 198.12 134.62 0)
 			(effects
@@
 			)
 		)
-		(property "Footprint" "Button_Switch_THT:SW_PUSH_6mm_H5mm"
+		(property "Footprint" "Button_Switch_THT:SW_PUSH_6mm_H6.5mm"
 			(at 261.62 134.62 0)
 			(effects
@@
 			)
 		)
-		(property "Footprint" "Button_Switch_THT:SW_PUSH_6mm_H5mm"
+		(property "Footprint" "Button_Switch_THT:SW_PUSH_6mm_H6.5mm"
 			(at 101.6 134.62 0)
 			(effects
@@
 			)
 		)
-		(property "Footprint" "Button_Switch_THT:SW_PUSH_6mm_H5mm"
+		(property "Footprint" "Button_Switch_THT:SW_PUSH_6mm_H6.5mm"
 			(at 172.72 134.62 0)
 			(effects
@@
 			)
 		)
-		(property "Footprint" "Button_Switch_THT:SW_PUSH_6mm_H5mm"
+		(property "Footprint" "Button_Switch_THT:SW_PUSH_6mm_H6.5mm"
 			(at 116.84 134.62 0)
 			(effects
@@
 			)
 		)
-		(property "Footprint" "Connector_Coaxial:SMA_BAT_Wireless_BWSMA-KWE-Z001"
+		(property "Footprint" "Connector_Coaxial:SMA_Connector_at_Honbu_3-1478978-1"
 			(at 76.2 116.84 0)
 			(effects
@@
 			)
 		)
-		(property "Footprint" "Button_Switch_THT:SW_PUSH_6mm_H5mm"
+		(property "Footprint" "Button_Switch_THT:SW_PUSH_6mm_H6.5mm"
 			(at 132.08 134.62 0)
 			(effects
@@
 			)
 		)
-		(property "Footprint" "Button_Switch_THT:SW_PUSH_6mm_H5mm"
+		(property "Footprint" "Button_Switch_THT:SW_PUSH_6mm_H6.5mm"
 			(at 210.82 134.62 0)
 			(effects
@@
 			)
 		)
-		(property "Footprint" "Button_Switch_THT:SW_PUSH_6mm_H5mm"
+		(property "Footprint" "Button_Switch_THT:SW_PUSH_6mm_H6.5mm"
 			(at 248.92 134.62 0)
 			(effects
@@
 			)
 		)
-		(property "Footprint" "Button_Switch_THT:SW_PUSH_6mm_H5mm"
+		(property "Footprint" "Button_Switch_THT:SW_PUSH_6mm_H6.5mm"
 			(at 185.42 134.62 0)
 			(effects
